Commit message: feat(): add kinematics

File: src/waregv_description/urdf/waregv.urdf.xacro (robot description, xacro)
@@ -7,5 +7,5 @@
     <link name="base_link">
         <inertial>
-            <origin xyz="0 0 0.045" rpy="0 0 0" />
+            <origin xyz="-0.08 0 0.045" rpy="0 0 0" />
             <mass value="3.0" />
             <inertia ixx="0.05625" ixy="0.0" ixz="0.0" iyy="0.05625" iyz="0.0" izz="0.10125" />
@@ -68,10 +68,10 @@
     <link name="wheel_front_right_link">
         <inertial>
-            <origin xyz="0 0 0" rpy="1.57 0 0" />
+            <origin xyz="0 0.015 0" rpy="1.57 0 0" />
             <mass value="0.25" />
             <inertia ixx="0.000138" ixy="0.0" ixz="0.0" iyy="0.000138" iyz="0.0" izz="0.000226" />
         </inertial>
         <visual>
-            <origin rpy="0 0 1.57" xyz="0 0.008 0" />
+            <origin rpy="0 0 1.57" xyz="0 -0.008 0" />
             <geometry>
                 <mesh filename="package://waregv_description/meshes/waregv_wheel.obj"
@@ -88,10 +88,10 @@
     <link name="wheel_rear_right_link">
         <inertial>
-            <origin xyz="0 0 0" rpy="1.57 0 0" />
+            <origin xyz="0 0.015 0" rpy="1.57 0 0" />
             <mass value="0.25" />
             <inertia ixx="0.000138" ixy="0.0" ixz="0.0" iyy="0.000138" iyz="0.0" izz="0.000226" />
         </inertial>
         <visual>
-            <origin rpy="0 0 1.57" xyz="0 0.008 0" />
+            <origin rpy="0 0 1.57" xyz="0 -0.008 0" />
             <geometry>
                 <mesh filename="package://waregv_description/meshes/waregv_wheel.obj"
@@ -168,5 +168,5 @@
         <parent link="base_link" />
         <child link="wheel_front_right_link" />
-        <origin rpy="0 0 0" xyz="0.14 -0.22 0" />
+        <origin rpy="0 0 0" xyz="0.14 -0.205 0" />
         <axis xyz="0 1 0" />
     </joint>
@@ -174,5 +174,5 @@
         <parent link="base_link" />
         <child link="wheel_rear_right_link" />
-        <origin rpy="0 0 0" xyz="-0.14 -0.22 0" />
+        <origin rpy="0 0 0" xyz="-0.14 -0.205 0" />
         <axis xyz="0 1 0" />
     </joint>

File: src/waregv_description/urdf/waregv_gazebo.xacro (robot description, xacro)
@@ -41,9 +41,29 @@
 </gazebo>
     <gazebo reference="base_link">
-        <sensor name="imu" type="imu">
+        <sensor name="imu_1" type="imu">
             <always_on>true</always_on>
             <update_rate>100</update_rate>
-            <topic>/imu</topic>
+            <topic>/imu_1</topic>
             <gz_frame_id>base_link</gz_frame_id>
+            <imu>
+                <angular_velocity>
+                    <x><noise type="gaussian"><mean>0.0</mean><stddev>2e-4</stddev></noise></x>
+                    <y><noise type="gaussian"><mean>0.0</mean><stddev>2e-4</stddev></noise></y>
+                    <z><noise type="gaussian"><mean>0.0</mean><stddev>2e-4</stddev></noise></z>
+                </angular_velocity>
+                <linear_acceleration>
+                    <x><noise type="gaussian"><mean>0.0</mean><stddev>1.7e-2</stddev></noise></x>
+                    <y><noise type="gaussian"><mean>0.0</mean><stddev>1.7e-2</stddev></noise></y>
+                    <z><noise type="gaussian"><mean>0.0</mean><stddev>1.7e-2</stddev></noise></z>
+                </linear_acceleration>
+            </imu>
+        </sensor>
+    </gazebo>
+    <gazebo reference="camera_link">
+        <sensor name="imu_2" type="imu">
+            <always_on>true</always_on>
+            <update_rate>100</update_rate>
+            <topic>/imu_2</topic>
+            <gz_frame_id>camera_link</gz_frame_id>
             <imu>
                 <angular_velocity>

Commit message: feat(): added new rover with slam

File: src/waregv_description/urdf/waregv.urdf.xacro (robot description, xacro)
@@ -7,19 +7,19 @@
     <link name="base_link">
         <inertial>
-            <origin xyz="-0.08 0 0.045" rpy="0 0 0" />
+            <origin xyz="-0.03 0 0" rpy="0 0 0" />
             <mass value="3.0" />
-            <inertia ixx="0.05625" ixy="0.0" ixz="0.0" iyy="0.05625" iyz="0.0" izz="0.10125" />
+            <inertia ixx="0.026282" ixy="0.0" ixz="0.0" iyy="0.026282" iyz="0.0" izz="0.045" />
         </inertial>
         <visual>
-            <origin rpy="1.57 0 1.57" xyz="0.2 0 0.045" />
+            <origin rpy="0 0 1.57" xyz="0 0 0" />
             <geometry>
-                <mesh filename="package://waregv_description/meshes/waregv_chasis.obj"
+                <mesh filename="package://waregv_description/meshes/waregv_v2_chasis.obj"
                     scale="0.01 0.01 0.01" />
             </geometry>
         </visual>
         <collision>
-            <origin rpy="1.57 0 1.57" xyz="0.2 0 0.045" />
+            <origin rpy="0 0 1.57" xyz="0 0 0" />
             <geometry>
-                <mesh filename="package://waregv_description/meshes/waregv_chasis.obj"
+                <mesh filename="package://waregv_description/meshes/waregv_v2_chasis.obj"
                     scale="0.01 0.01 0.01" />
             </geometry>
@@ -28,12 +28,12 @@
     <link name="wheel_front_left_link">
         <inertial>
-            <origin xyz="0 0 0" rpy="1.57 0 0" />
+            <origin xyz="0 0 0" rpy="0 0 1.57" />
             <mass value="0.25" />
-            <inertia ixx="0.000138" ixy="0.0" ixz="0.0" iyy="0.000138" iyz="0.0" izz="0.000226" />
+            <inertia ixx="0.0013681" ixy="0.0" ixz="0.0" iyy="0.0013681" iyz="0.0" izz="0.000132" />
         </inertial>
         <visual>
-            <origin rpy="0 0 -1.57" xyz="0 0.008 0" />
+            <origin rpy="0 0 1.57" xyz="0 0 0" />
             <geometry>
-                <mesh filename="package://waregv_description/meshes/waregv_wheel.obj"
+                <mesh filename="package://waregv_description/meshes/wheel.obj"
                     scale="0.01 0.01 0.01" />
             </geometry>
@@ -42,5 +42,5 @@
             <origin xyz="0 0 0" rpy="1.57 0 0" />
             <geometry>
-                <cylinder length="0.035" radius="0.0425" />
+                <cylinder length="0.025" radius="0.0325" />
             </geometry>
         </collision>
@@ -48,12 +48,12 @@
     <link name="wheel_rear_left_link">
         <inertial>
-            <origin xyz="0 0 0" rpy="1.57 0 0" />
+            <origin xyz="0 0 0" rpy="0 0 1.57" />
             <mass value="0.25" />
-            <inertia ixx="0.000138" ixy="0.0" ixz="0.0" iyy="0.000138" iyz="0.0" izz="0.000226" />
+            <inertia ixx="0.0013681" ixy="0.0" ixz="0.0" iyy="0.0013681" iyz="0.0" izz="0.000132" />
         </inertial>
         <visual>
-            <origin rpy="0 0 -1.57" xyz="0 0.008 0" />
+            <origin rpy="0 0 1.57" xyz="0 0 0" />
             <geometry>
-                <mesh filename="package://waregv_description/meshes/waregv_wheel.obj"
+                <mesh filename="package://waregv_description/meshes/wheel.obj"
                     scale="0.01 0.01 0.01" />
             </geometry>
@@ -62,5 +62,5 @@
             <origin xyz="0 0 0" rpy="1.57 0 0" />
             <geometry>
-                <cylinder length="0.035" radius="0.0425" />
+                <cylinder length="0.025" radius="0.0325" />
             </geometry>
         </collision>
@@ -68,12 +68,12 @@
     <link name="wheel_front_right_link">
         <inertial>
-            <origin xyz="0 0.015 0" rpy="1.57 0 0" />
+            <origin xyz="0 0 0" rpy="0 0 1.57" />
             <mass value="0.25" />
-            <inertia ixx="0.000138" ixy="0.0" ixz="0.0" iyy="0.000138" iyz="0.0" izz="0.000226" />
+            <inertia ixx="0.0013681" ixy="0.0" ixz="0.0" iyy="0.0013681" iyz="0.0" izz="0.000132" />
         </inertial>
         <visual>
-            <origin rpy="0 0 1.57" xyz="0 -0.008 0" />
+            <origin rpy="0 0 -1.57" xyz="0 0 0" />
             <geometry>
-                <mesh filename="package://waregv_description/meshes/waregv_wheel.obj"
+                <mesh filename="package://waregv_description/meshes/wheel.obj"
                     scale="0.01 0.01 0.01" />
             </geometry>
@@ -82,5 +82,5 @@
             <origin xyz="0 0 0" rpy="1.57 0 0" />
             <geometry>
-                <cylinder length="0.035" radius="0.0425" />
+                <cylinder length="0.025" radius="0.0325" />
             </geometry>
         </collision>
@@ -88,12 +88,12 @@
     <link name="wheel_rear_right_link">
         <inertial>
-            <origin xyz="0 0.015 0" rpy="1.57 0 0" />
+            <origin xyz="0 0 0" rpy="0 0 1.57" />
             <mass value="0.25" />
-            <inertia ixx="0.000138" ixy="0.0" ixz="0.0" iyy="0.000138" iyz="0.0" izz="0.000226" />
+            <inertia ixx="0.0013681" ixy="0.0" ixz="0.0" iyy="0.0013681" iyz="0.0" izz="0.000132" />
         </inertial>
         <visual>
-            <origin rpy="0 0 1.57" xyz="0 -0.008 0" />
+            <origin rpy="0 0 -1.57" xyz="0 0 0" />
             <geometry>
-                <mesh filename="package://waregv_description/meshes/waregv_wheel.obj"
+                <mesh filename="package://waregv_description/meshes/wheel.obj"
                     scale="0.01 0.01 0.01" />
             </geometry>
@@ -102,5 +102,5 @@
             <origin xyz="0 0 0" rpy="1.57 0 0" />
             <geometry>
-                <cylinder length="0.035" radius="0.0425" />
+                <cylinder length="0.025" radius="0.0325" />
             </geometry>
         </collision>
@@ -108,7 +108,7 @@
     <link name="camera_link">
         <inertial>
+            <mass value="0.072" />
             <origin xyz="0 0 0" rpy="0 0 0" />
-            <mass value="0.5" />
-            <inertia ixx="0.001004" ixy="0.0" ixz="0.0" iyy="0.000133" iyz="0.0" izz="0.001004" />
+            <inertia ixx="0.0000075" ixy="0.0" ixz="0.0" iyy="0.0000522" iyz="0.0" izz="0.0000522" />
         </inertial>
         <visual>
@@ -122,26 +122,12 @@
     <link name="lidar_link">
         <inertial>
+            <mass value="0.170" />
             <origin xyz="0 0 0" rpy="0 0 0" />
-            <mass value="0.3" />
-            <inertia ixx="0.000185" ixy="0.0" ixz="0.0" iyy="0.000185" iyz="0.0" izz="0.000245" />
+            <inertia ixx="0.0001131" ixy="0.0" ixz="0.0" iyy="0.0001755" iyz="0.0" izz="0.0002025" />
         </inertial>
         <visual>
-            <origin rpy="1.57 0 0" xyz="0 0 0" />
+            <origin rpy="1.57 0 3.14" xyz="0 0 0" />
             <geometry>
-                <mesh filename="package://waregv_description/meshes/waregv_lidar.obj"
-                    scale="0.01 0.01 0.01" />
-            </geometry>
-        </visual>
-    </link>
-    <link name="sonar_link">
-        <inertial>
-            <origin xyz="0 0 0" rpy="0 0 0" />
-            <mass value="0.05" />
-            <inertia ixx="0.000012" ixy="0.0" ixz="0.0" iyy="0.000003" iyz="0.0" izz="0.000012" />
-        </inertial>
-        <visual>
-            <origin rpy="1.57  0 1.57" xyz="0 0 0" />
-            <geometry>
-                <mesh filename="package://waregv_description/meshes/waregv_ultrasonic_sensor.obj"
+                <mesh filename="package://waregv_description/meshes/lidar.obj"
                     scale="0.01 0.01 0.01" />
             </geometry>
@@ -156,5 +142,5 @@
         <parent link="base_link" />
         <child link="wheel_front_left_link" />
-        <origin rpy="0 0 0" xyz="0.14 0.205 0" />
+        <origin rpy="0 0 0" xyz="0.09 0.088 -0.01" />
         <axis xyz="0 1 0" />
     </joint>
@@ -162,5 +148,5 @@
         <parent link="base_link" />
         <child link="wheel_rear_left_link" />
-        <origin rpy="0 0 0" xyz="-0.14 0.205 0" />
+        <origin rpy="0 0 0" xyz="-0.09 0.088 -0.01" />
         <axis xyz="0 1 0" />
     </joint>
@@ -168,5 +154,5 @@
         <parent link="base_link" />
         <child link="wheel_front_right_link" />
-        <origin rpy="0 0 0" xyz="0.14 -0.205 0" />
+        <origin rpy="0 0 0" xyz="0.09 -0.088 -0.01" />
         <axis xyz="0 1 0" />
     </joint>
@@ -174,5 +160,5 @@
         <parent link="base_link" />
         <child link="wheel_rear_right_link" />
-        <origin rpy="0 0 0" xyz="-0.14 -0.205 0" />
+        <origin rpy="0 0 0" xyz="-0.09 -0.088 -0.01" />
         <axis xyz="0 1 0" />
     </joint>
@@ -180,15 +166,10 @@
         <parent link="base_link" />
         <child link="camera_link" />
-        <origin rpy="0 0 0" xyz="0.242 0 0.265" />
+        <origin rpy="0 0 0" xyz="0.14 -0.002 0.098" />
     </joint>
     <joint name="lidar_joint" type="fixed">
         <parent link="base_link" />
         <child link="lidar_link" />
-        <origin rpy="0 0 0" xyz="0.2275 0 0.33" />
-    </joint>
-    <joint name="sonar_joint" type="fixed">
-        <parent link="base_link" />
-        <child link="sonar_link" />
-        <origin rpy="0 0 0" xyz="0.228 0 0.037" />
+        <origin rpy="0 0 0" xyz="0.095 0 0.155" />
     </joint>
 </robot>

File: src/waregv_description/urdf/waregv_gazebo.xacro (robot description, xacro)
@@ -82,4 +82,5 @@
     <gazebo reference="lidar_link">
         <sensor name="gpu_lidar" type="gpu_lidar">
+             <pose>0 0 0 0 0 0</pose>
             <update_rate>10</update_rate>
             <topic>/scan</topic>
@@ -110,28 +111,4 @@
         </sensor>
     </gazebo>
-    <gazebo reference="sonar_link">
-        <sensor name="sonar_lidar" type="gpu_lidar">
-            <update_rate>20</update_rate>
-            <topic>/sonar_scan</topic>
-            <always_on>true</always_on>
-            <visualize>true</visualize>
-            <gz_frame_id>sonar_link</gz_frame_id>
-            <lidar>
-                <scan>
-                    <horizontal>
-                        <samples>15</samples>
-                        <resolution>1</resolution>
-                        <min_angle>-0.1</min_angle>
-                        <max_angle>0.1</max_angle>
-                    </horizontal>
-                </scan>
-                <range>
-                    <min>0.05</min>
-                    <max>3.0</max>
-                    <resolution>0.01</resolution>
-                </range>
-            </lidar>
-        </sensor>
-    </gazebo>
     <gazebo reference="camera_link">
         <sensor name="camera" type="camera">

Commit message: feat(): add simuntanous slam and nav

File: src/waregv_description/urdf/waregv.urdf.xacro (robot description, xacro)
@@ -143,4 +143,6 @@
         <child link="wheel_front_left_link" />
         <origin rpy="0 0 0" xyz="0.09 0.088 -0.01" />
+        <limit effort="10.0" velocity="45.0" />
+        <dynamics damping="0.05" friction="0.05" />
         <axis xyz="0 1 0" />
     </joint>
@@ -149,4 +151,6 @@
         <child link="wheel_rear_left_link" />
         <origin rpy="0 0 0" xyz="-0.09 0.088 -0.01" />
+        <limit effort="10.0" velocity="45.0" />
+        <dynamics damping="0.05" friction="0.05" />
         <axis xyz="0 1 0" />
     </joint>
@@ -155,4 +159,6 @@
         <child link="wheel_front_right_link" />
         <origin rpy="0 0 0" xyz="0.09 -0.088 -0.01" />
+        <limit effort="10.0" velocity="45.0" />
+        <dynamics damping="0.05" friction="0.05" />
         <axis xyz="0 1 0" />
     </joint>
@@ -161,4 +167,6 @@
         <child link="wheel_rear_right_link" />
         <origin rpy="0 0 0" xyz="-0.09 -0.088 -0.01" />
+        <limit effort="10.0" velocity="45.0" />
+        <dynamics damping="0.05" friction="0.05" />
         <axis xyz="0 1 0" />
     </joint>

File: src/waregv_description/urdf/waregv_ros2_control.xacro (robot description, xacro)
@@ -7,6 +7,6 @@
         <joint name="wheel_front_right_joint">
             <command_interface name="velocity">
-                <param name="min">-1</param>
-                <param name="max">1</param>
+                <param name="min">-40</param>
+<param name="max">40</param>
             </command_interface>
             <state_interface name="position" />
@@ -15,6 +15,6 @@
         <joint name="wheel_front_left_joint">
             <command_interface name="velocity">
-                <param name="min">-1</param>
-                <param name="max">1</param>
+                <param name="min">-40</param>
+<param name="max">40</param>
             </command_interface>
             <state_interface name="position" />
@@ -23,6 +23,6 @@
         <joint name="wheel_rear_right_joint">
             <command_interface name="velocity">
-                <param name="min">-1</param>
-                <param name="max">1</param>
+                <param name="min">-40</param>
+<param name="max">40</param>
             </command_interface>
             <state_interface name="position" />
@@ -31,6 +31,6 @@
         <joint name="wheel_rear_left_joint">
             <command_interface name="velocity">
-                <param name="min">-1</param>
-                <param name="max">1</param>
+                <param name="min">-40</param>
+<param name="max">40</param>
             </command_interface>
             <state_interface name="position" />

Commit message: feat(): added waregv_v2 with nav

File: src/waregv_description/urdf/waregv.urdf.xacro (robot description, xacro)
@@ -12,5 +12,5 @@
         </inertial>
         <visual>
-            <origin rpy="0 0 1.57" xyz="0 0 0" />
+            <origin rpy="1.57 0 1.57" xyz="0.03 0 0.015" />
             <geometry>
                 <mesh filename="package://waregv_description/meshes/waregv_v2_chasis.obj"
@@ -19,5 +19,5 @@
         </visual>
         <collision>
-            <origin rpy="0 0 1.57" xyz="0 0 0" />
+             <origin rpy="1.57 0 1.57" xyz="0.03 0 0.015" />
             <geometry>
                 <mesh filename="package://waregv_description/meshes/waregv_v2_chasis.obj"
@@ -30,10 +30,10 @@
             <origin xyz="0 0 0" rpy="0 0 1.57" />
             <mass value="0.25" />
-            <inertia ixx="0.0013681" ixy="0.0" ixz="0.0" iyy="0.0013681" iyz="0.0" izz="0.000132" />
+            <inertia ixx="0.0000953" ixy="0.0" ixz="0.0" iyy="0.0000953" iyz="0.0" izz="0.0001531" />
         </inertial>
         <visual>
             <origin rpy="0 0 1.57" xyz="0 0 0" />
             <geometry>
-                <mesh filename="package://waregv_description/meshes/wheel.obj"
+                <mesh filename="package://waregv_description/meshes/waregv_v2_wheel.obj"
                     scale="0.01 0.01 0.01" />
             </geometry>
@@ -42,5 +42,5 @@
             <origin xyz="0 0 0" rpy="1.57 0 0" />
             <geometry>
-                <cylinder length="0.025" radius="0.0325" />
+                <cylinder length="0.030" radius="0.035" />
             </geometry>
         </collision>
@@ -50,10 +50,10 @@
             <origin xyz="0 0 0" rpy="0 0 1.57" />
             <mass value="0.25" />
-            <inertia ixx="0.0013681" ixy="0.0" ixz="0.0" iyy="0.0013681" iyz="0.0" izz="0.000132" />
+           <inertia ixx="0.0000953" ixy="0.0" ixz="0.0" iyy="0.0000953" iyz="0.0" izz="0.0001531" />
         </inertial>
         <visual>
             <origin rpy="0 0 1.57" xyz="0 0 0" />
             <geometry>
-                <mesh filename="package://waregv_description/meshes/wheel.obj"
+                <mesh filename="package://waregv_description/meshes/waregv_v2_wheel.obj"
                     scale="0.01 0.01 0.01" />
             </geometry>
@@ -62,5 +62,5 @@
             <origin xyz="0 0 0" rpy="1.57 0 0" />
             <geometry>
-                <cylinder length="0.025" radius="0.0325" />
+                <cylinder length="0.030" radius="0.035" />
             </geometry>
         </collision>
@@ -70,10 +70,10 @@
             <origin xyz="0 0 0" rpy="0 0 1.57" />
             <mass value="0.25" />
-            <inertia ixx="0.0013681" ixy="0.0" ixz="0.0" iyy="0.0013681" iyz="0.0" izz="0.000132" />
+            <inertia ixx="0.0000953" ixy="0.0" ixz="0.0" iyy="0.0000953" iyz="0.0" izz="0.0001531" />
         </inertial>
         <visual>
             <origin rpy="0 0 -1.57" xyz="0 0 0" />
             <geometry>
-                <mesh filename="package://waregv_description/meshes/wheel.obj"
+                <mesh filename="package://waregv_description/meshes/waregv_v2_wheel.obj"
                     scale="0.01 0.01 0.01" />
             </geometry>
@@ -82,5 +82,5 @@
             <origin xyz="0 0 0" rpy="1.57 0 0" />
             <geometry>
-                <cylinder length="0.025" radius="0.0325" />
+                <cylinder length="0.030" radius="0.035" />
             </geometry>
         </collision>
@@ -90,10 +90,10 @@
             <origin xyz="0 0 0" rpy="0 0 1.57" />
             <mass value="0.25" />
-            <inertia ixx="0.0013681" ixy="0.0" ixz="0.0" iyy="0.0013681" iyz="0.0" izz="0.000132" />
+            <inertia ixx="0.0000953" ixy="0.0" ixz="0.0" iyy="0.0000953" iyz="0.0" izz="0.0001531" />
         </inertial>
         <visual>
             <origin rpy="0 0 -1.57" xyz="0 0 0" />
             <geometry>
-                <mesh filename="package://waregv_description/meshes/wheel.obj"
+                <mesh filename="package://waregv_description/meshes/waregv_v2_wheel.obj"
                     scale="0.01 0.01 0.01" />
             </geometry>
@@ -102,5 +102,5 @@
             <origin xyz="0 0 0" rpy="1.57 0 0" />
             <geometry>
-                <cylinder length="0.025" radius="0.0325" />
+                <cylinder length="0.030" radius="0.035" />
             </geometry>
         </collision>
@@ -124,5 +124,5 @@
             <mass value="0.170" />
             <origin xyz="0 0 0" rpy="0 0 0" />
-            <inertia ixx="0.0001131" ixy="0.0" ixz="0.0" iyy="0.0001755" iyz="0.0" izz="0.0002025" />
+            <inertia ixx="0.0001131" ixy="0.0" ixz="0.0" iyy="0.0001755" iyz="0.0" izz="0.0002030" />
         </inertial>
         <visual>
@@ -166,10 +166,10 @@
         <parent link="base_link" />
         <child link="camera_link" />
-        <origin rpy="0 0 0" xyz="0.14 -0.002 0.098" />
+        <origin rpy="0 0 0" xyz="0.133 -0.002 0.075" />
     </joint>
     <joint name="lidar_joint" type="fixed">
         <parent link="base_link" />
         <child link="lidar_link" />
-        <origin rpy="0 0 0" xyz="0.095 0 0.155" />
+        <origin rpy="0 0 0" xyz="0.095 0 0.12" />
     </joint>
 </robot>
