Commit message: feat(): add foxglove

File: src/waregv_description/urdf/waregv.urdf.xacro (robot description, xacro)
@@ -33,5 +33,5 @@
         </inertial>
         <visual>
-            <origin rpy="0 0 1.57" xyz="0 0 0" />
+            <origin rpy="0 0 -1.57" xyz="0 0 0" />
             <geometry>
                 <mesh filename="package://waregv_description/meshes/waregv_v2_wheel.obj"
@@ -53,5 +53,5 @@
         </inertial>
         <visual>
-            <origin rpy="0 0 1.57" xyz="0 0 0" />
+            <origin rpy="0 0 -1.57" xyz="0 0 0" />
             <geometry>
                 <mesh filename="package://waregv_description/meshes/waregv_v2_wheel.obj"
@@ -73,5 +73,5 @@
         </inertial>
         <visual>
-            <origin rpy="0 0 -1.57" xyz="0 0 0" />
+            <origin rpy="0 0 1.57" xyz="0 0 0" />
             <geometry>
                 <mesh filename="package://waregv_description/meshes/waregv_v2_wheel.obj"
@@ -93,5 +93,5 @@
         </inertial>
         <visual>
-            <origin rpy="0 0 -1.57" xyz="0 0 0" />
+            <origin rpy="0 0 1.57" xyz="0 0 0" />
             <geometry>
                 <mesh filename="package://waregv_description/meshes/waregv_v2_wheel.obj"
@@ -142,32 +142,32 @@
         <parent link="base_link" />
         <child link="wheel_front_left_link" />
-        <origin rpy="0 0 0" xyz="0.09 0.088 -0.01" />
+        <origin rpy="0 0 3.14" xyz="0.09 0.088 -0.01" />
         <limit effort="10.0" velocity="45.0" />
         <dynamics damping="0.05" friction="0.05" />
-        <axis xyz="0 1 0" />
+        <axis xyz="0 -1 0" />
     </joint>
     <joint name="wheel_rear_left_joint" type="continuous">
         <parent link="base_link" />
         <child link="wheel_rear_left_link" />
-        <origin rpy="0 0 0" xyz="-0.09 0.088 -0.01" />
+        <origin rpy="0 0 3.14" xyz="-0.09 0.088 -0.01" />
         <limit effort="10.0" velocity="45.0" />
         <dynamics damping="0.05" friction="0.05" />
-        <axis xyz="0 1 0" />
+        <axis xyz="0 -1 0" />
     </joint>
     <joint name="wheel_front_right_joint" type="continuous">
         <parent link="base_link" />
         <child link="wheel_front_right_link" />
-        <origin rpy="0 0 0" xyz="0.09 -0.088 -0.01" />
+        <origin rpy="0 0 3.14" xyz="0.09 -0.088 -0.01" />
         <limit effort="10.0" velocity="45.0" />
         <dynamics damping="0.05" friction="0.05" />
-        <axis xyz="0 1 0" />
+        <axis xyz="0 -1 0" />
     </joint>
     <joint name="wheel_rear_right_joint" type="continuous">
         <parent link="base_link" />
         <child link="wheel_rear_right_link" />
-        <origin rpy="0 0 0" xyz="-0.09 -0.088 -0.01" />
+        <origin rpy="0 0 3.14" xyz="-0.09 -0.088 -0.01" />
         <limit effort="10.0" velocity="45.0" />
         <dynamics damping="0.05" friction="0.05" />
-        <axis xyz="0 1 0" />
+        <axis xyz="0 -1 0" />
     </joint>
     <joint name="camera_joint" type="fixed">

File: src/waregv_description/urdf/waregv_gazebo.xacro (robot description, xacro)
@@ -41,8 +41,8 @@
 </gazebo>
     <gazebo reference="base_link">
-        <sensor name="imu_1" type="imu">
+        <sensor name="imu" type="imu">
             <always_on>true</always_on>
             <update_rate>100</update_rate>
-            <topic>/imu_1</topic>
+            <topic>/imu</topic>
             <gz_frame_id>base_link</gz_frame_id>
             <imu>

Commit message: minimize and add ros2 control with robot localization

File: src/waregv_description/urdf/waregv.urdf.xacro (robot description, xacro)
@@ -1,5 +1,4 @@
 <?xml version="1.0" encoding="UTF-8"?>
 <robot xmlns:xacro="http://www.ros.org/wiki/xacro" name="waregv">
-    <xacro:arg name="is_ignition" default="true" />
     <xacro:include filename="$(find waregv_description)/urdf/waregv_gazebo.xacro" />
     <xacro:include filename="$(find waregv_description)/urdf/waregv_ros2_control.xacro" />
@@ -14,13 +13,11 @@
             <origin rpy="1.57 0 1.57" xyz="0.03 0 0.015" />
             <geometry>
-                <mesh filename="package://waregv_description/meshes/waregv_v2_chasis.obj"
-                    scale="0.01 0.01 0.01" />
+                <mesh filename="package://waregv_description/meshes/chasis.obj" scale="0.01 0.01 0.01" />
             </geometry>
         </visual>
         <collision>
-             <origin rpy="1.57 0 1.57" xyz="0.03 0 0.015" />
+            <origin rpy="1.57 0 1.57" xyz="0.03 0 0.015" />
             <geometry>
-                <mesh filename="package://waregv_description/meshes/waregv_v2_chasis.obj"
-                    scale="0.01 0.01 0.01" />
+                <mesh filename="package://waregv_description/meshes/chasis.obj" scale="0.01 0.01 0.01" />
             </geometry>
         </collision>
@@ -35,6 +32,5 @@
             <origin rpy="0 0 -1.57" xyz="0 0 0" />
             <geometry>
-                <mesh filename="package://waregv_description/meshes/waregv_v2_wheel.obj"
-                    scale="0.01 0.01 0.01" />
+                <mesh filename="package://waregv_description/meshes/wheel.obj" scale="0.01 0.01 0.01" />
             </geometry>
         </visual>
@@ -50,11 +46,10 @@
             <origin xyz="0 0 0" rpy="0 0 1.57" />
             <mass value="0.25" />
-           <inertia ixx="0.0000953" ixy="0.0" ixz="0.0" iyy="0.0000953" iyz="0.0" izz="0.0001531" />
+            <inertia ixx="0.0000953" ixy="0.0" ixz="0.0" iyy="0.0000953" iyz="0.0" izz="0.0001531" />
         </inertial>
         <visual>
             <origin rpy="0 0 -1.57" xyz="0 0 0" />
             <geometry>
-                <mesh filename="package://waregv_description/meshes/waregv_v2_wheel.obj"
-                    scale="0.01 0.01 0.01" />
+                <mesh filename="package://waregv_description/meshes/wheel.obj" scale="0.01 0.01 0.01" />
             </geometry>
         </visual>
@@ -75,6 +70,5 @@
             <origin rpy="0 0 1.57" xyz="0 0 0" />
             <geometry>
-                <mesh filename="package://waregv_description/meshes/waregv_v2_wheel.obj"
-                    scale="0.01 0.01 0.01" />
+                <mesh filename="package://waregv_description/meshes/wheel.obj" scale="0.01 0.01 0.01" />
             </geometry>
         </visual>
@@ -95,6 +89,5 @@
             <origin rpy="0 0 1.57" xyz="0 0 0" />
             <geometry>
-                <mesh filename="package://waregv_description/meshes/waregv_v2_wheel.obj"
-                    scale="0.01 0.01 0.01" />
+                <mesh filename="package://waregv_description/meshes/wheel.obj" scale="0.01 0.01 0.01" />
             </geometry>
         </visual>
@@ -115,6 +108,5 @@
             <origin rpy="1.57 0 1.57" xyz="0 0 0" />
             <geometry>
-                <mesh filename="package://waregv_description/meshes/waregv_depth_camera.obj"
-                    scale="0.01 0.01 0.01" />
+                <mesh filename="package://waregv_description/meshes/camera.obj" scale="0.01 0.01 0.01" />
             </geometry>
         </visual>
@@ -129,6 +121,5 @@
             <origin rpy="1.57 0 3.14" xyz="0 0 0" />
             <geometry>
-                <mesh filename="package://waregv_description/meshes/lidar.obj"
-                    scale="0.01 0.01 0.01" />
+                <mesh filename="package://waregv_description/meshes/lidar.obj" scale="0.01 0.01 0.01" />
             </geometry>
         </visual>

File: src/waregv_description/urdf/waregv_gazebo.xacro (robot description, xacro)
@@ -1,5 +1,20 @@
 <?xml version="1.0" encoding="UTF-8"?>
 <robot xmlns:xacro="http://ros.org" name="waregv">
+    <gazebo>
+        <plugin filename="gz_ros2_control-system" name="gz_ros2_control::GazeboSimROS2ControlPlugin">
+            <parameters>$(find waregv_description)/config/controller.yaml</parameters>
+        </plugin>
+        <plugin filename="gz-sim-imu-system" name="gz::sim::systems::Imu"/>
+        <plugin filename="gz-sim-sensors-system" name="gz::sim::systems::Sensors"/>
+    </gazebo>
     <gazebo reference="wheel_front_left_link">
+        <mu1>2.5</mu1>
+        <mu2>2.5</mu2>
+        <kp>1000000.0</kp>
+        <kd>10.0</kd>
+        <minDepth>0.001</minDepth>
+        <maxVel>0.1</maxVel>
+    </gazebo>
+    <gazebo reference="wheel_front_right_link">
         <mu1>2.5</mu1>
         <mu2>2.5</mu2>
@@ -17,12 +32,4 @@
         <maxVel>0.1</maxVel>
     </gazebo>
-    <gazebo reference="wheel_front_right_link">
-        <mu1>2.5</mu1>
-        <mu2>2.5</mu2>
-        <kp>1000000.0</kp>
-        <kd>10.0</kd>
-        <minDepth>0.001</minDepth>
-        <maxVel>0.1</maxVel>
-    </gazebo>
     <gazebo reference="wheel_rear_right_link">
         <mu1>2.5</mu1>
@@ -33,11 +40,4 @@
         <maxVel>0.1</maxVel>
     </gazebo>
-   <gazebo>
-    <plugin filename="gz_ros2_control-system" name="gz_ros2_control::GazeboSimROS2ControlPlugin">
-        <parameters>$(find waregv_bringup)/config/controller.yaml</parameters>
-    </plugin>
-    <plugin filename="gz-sim-imu-system" name="gz::sim::systems::Imu"></plugin>
-    <plugin filename="gz-sim-sensors-system" name="gz::sim::systems::Sensors"></plugin>
-</gazebo>
     <gazebo reference="base_link">
         <sensor name="imu" type="imu">
@@ -60,32 +60,11 @@
         </sensor>
     </gazebo>
-    <gazebo reference="camera_link">
-        <sensor name="imu_camera" type="imu">
-            <always_on>true</always_on>
-            <update_rate>100</update_rate>
-            <topic>/imu_camera</topic>
-            <gz_frame_id>camera_link</gz_frame_id>
-            <imu>
-                <angular_velocity>
-                    <x><noise type="gaussian"><mean>0.0</mean><stddev>2e-4</stddev></noise></x>
-                    <y><noise type="gaussian"><mean>0.0</mean><stddev>2e-4</stddev></noise></y>
-                    <z><noise type="gaussian"><mean>0.0</mean><stddev>2e-4</stddev></noise></z>
-                </angular_velocity>
-                <linear_acceleration>
-                    <x><noise type="gaussian"><mean>0.0</mean><stddev>1.7e-2</stddev></noise></x>
-                    <y><noise type="gaussian"><mean>0.0</mean><stddev>1.7e-2</stddev></noise></y>
-                    <z><noise type="gaussian"><mean>0.0</mean><stddev>1.7e-2</stddev></noise></z>
-                </linear_acceleration>
-            </imu>
-        </sensor>
-    </gazebo>
     <gazebo reference="lidar_link">
         <sensor name="gpu_lidar" type="gpu_lidar">
-             <pose>0 0 0 0 0 0</pose>
+            <pose>0 0 0 0 0 0</pose>
             <update_rate>10</update_rate>
             <topic>/scan</topic>
             <always_on>true</always_on>
             <visualize>true</visualize>
-            <!-- Fixed for Gazebo Harmonic -->
             <gz_frame_id>lidar_link</gz_frame_id>
             <lidar>
@@ -113,5 +92,5 @@
     <gazebo reference="camera_link">
         <sensor name="camera" type="camera">
-             <pose>0 0 0 0 0 -0.1</pose>
+            <pose>0 0 0 0 0 -0.1</pose>
             <update_rate>30</update_rate>
             <topic>/camera/image_raw</topic>
@@ -120,5 +99,4 @@
             <gz_frame_id>camera_link</gz_frame_id>
             <camera>
-                <!-- D435i RGB horizontal FOV is exactly 69.4 degrees -->
                 <horizontal_fov>1.211258</horizontal_fov>
                 <image>
@@ -133,4 +111,22 @@
             </camera>
         </sensor>
+        <sensor name="imu_camera" type="imu">
+            <always_on>true</always_on>
+            <update_rate>100</update_rate>
+            <topic>/imu_camera</topic>
+            <gz_frame_id>camera_link</gz_frame_id>
+            <imu>
+                <angular_velocity>
+                    <x><noise type="gaussian"><mean>0.0</mean><stddev>2e-4</stddev></noise></x>
+                    <y><noise type="gaussian"><mean>0.0</mean><stddev>2e-4</stddev></noise></y>
+                    <z><noise type="gaussian"><mean>0.0</mean><stddev>2e-4</stddev></noise></z>
+                </angular_velocity>
+                <linear_acceleration>
+                    <x><noise type="gaussian"><mean>0.0</mean><stddev>1.7e-2</stddev></noise></x>
+                    <y><noise type="gaussian"><mean>0.0</mean><stddev>1.7e-2</stddev></noise></y>
+                    <z><noise type="gaussian"><mean>0.0</mean><stddev>1.7e-2</stddev></noise></z>
+                </linear_acceleration>
+            </imu>
+        </sensor>
     </gazebo>
 </robot>

File: src/waregv_description/urdf/waregv_ros2_control.xacro (robot description, xacro)
@@ -1,12 +1,21 @@
 <?xml version="1.0" encoding="UTF-8"?>
-<robot xmlns:xacro="http://www.ros.org/wiki/xacro" name="waregv">
+<robot xmlns:xacro="http://ros.org" name="waregv">
+    <xacro:arg name="sim_mode" default="false" />
     <ros2_control name="WareGVSystem" type="system">
         <hardware>
-            <plugin>gz_ros2_control/GazeboSimSystem</plugin>
+            <xacro:if value="$(arg sim_mode)">
+                <plugin>gz_ros2_control/GazeboSimSystem</plugin>
+            </xacro:if>
+            <xacro:unless value="$(arg sim_mode)">
+                <plugin>waregv_hardware/STS3215ServoControlDriver</plugin>
+                <param name="port_left">/dev/ttyAMA2</param>
+                <param name="port_right">/dev/ttyAMA3</param>
+                <param name="baud_rate">1000000</param>
+            </xacro:unless>
         </hardware>
         <joint name="wheel_front_right_joint">
             <command_interface name="velocity">
-                <param name="min">-40</param>
-<param name="max">40</param>
+                <param name="min">-9</param>
+                <param name="max">9</param>
             </command_interface>
             <state_interface name="position" />
@@ -15,6 +24,6 @@
         <joint name="wheel_front_left_joint">
             <command_interface name="velocity">
-                <param name="min">-40</param>
-<param name="max">40</param>
+                <param name="min">-9</param>
+                <param name="max">9</param>
             </command_interface>
             <state_interface name="position" />
@@ -23,6 +32,6 @@
         <joint name="wheel_rear_right_joint">
             <command_interface name="velocity">
-                <param name="min">-40</param>
-<param name="max">40</param>
+                <param name="min">-9</param>
+                <param name="max">9</param>
             </command_interface>
             <state_interface name="position" />
@@ -31,6 +40,6 @@
         <joint name="wheel_rear_left_joint">
             <command_interface name="velocity">
-                <param name="min">-40</param>
-<param name="max">40</param>
+                <param name="min">-9</param>
+                <param name="max">9</param>
             </command_interface>
             <state_interface name="position" />
